File: BaselineRP2040MotorController/RaspberryPiPico.kicad_sch (KiCad schematic)
At the start: 33 parts, among them J1 CPU1 USB, J5 Conn_01x06, SW1 KT11B2SAM34LFS, U1 USBLC6-4SC6, U2 W25Q128JVSIQ, U3 RP2040, U4 USBLC6-2P6, Y1 12MHz

Commit message: Drop some features.
Parts:
- D1: footprint Diode_THT:D_DO-201AD_P15.24mm_Horizontal -> Diode_SMD:D_SOD-123
- J5: footprint Connector_PinHeader_2.54mm:PinHeader_1x06_P2.54mm_Vertical -> Connector_PinHeader_2.00mm:PinHeader_1x06_P2.00mm_Vertical
- SW1: footprint Button_Switch_SMD:SW_SPST_Omron_B3FS-100xP -> Button_Switch_THT:SW_PUSH_6mm_H9.5mm
Changed lines of the file:
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@@
 			)
 		)
-		(property "Footprint" "Button_Switch_SMD:SW_SPST_Omron_B3FS-100xP"
+		(property "Footprint" "Button_Switch_THT:SW_PUSH_6mm_H9.5mm"
 			(at 48.26 58.42 0)
 			(effects
@@
 			)
 		)
-		(property "Footprint" "Connector_PinHeader_2.54mm:PinHeader_1x06_P2.54mm_Vertical"
+		(property "Footprint" "Connector_PinHeader_2.00mm:PinHeader_1x06_P2.00mm_Vertical"
 			(at 110.49 148.59 0)
 			(effects
@@
 			)
 		)
-		(property "Footprint" "Diode_THT:D_DO-201AD_P15.24mm_Horizontal"
+		(property "Footprint" "Diode_SMD:D_SOD-123"
 			(at 73.66 86.995 0)
 			(effects

Commit message: Just before dropping the self build of the 2040
Connections:
- net GND: now also J1.A8 (SBU1), J1.B8 (SBU2), U2.4 (GND)
