File: BaselineRP2040MotorController/PowerFiltering.kicad_sch (KiCad schematic)
At the start: 22 parts, among them U13 TX4139

Commit message: Heh - Super cut down.
Parts:
- removed C49: 47uF 63V solid, Capacitor_SMD:CP_Elec_8x10.5, symbol Device:C_Polarized
- removed C51, C64, C65: 4.7uF 100V, Capacitor_SMD:C_1210_3225Metric, symbol Device:C
- removed C52: 100nF 100V, Capacitor_SMD:C_0805_2012Metric, symbol Device:C
- removed C55: 100n, Capacitor_SMD:C_0603_1608Metric, symbol Device:C
- removed C57: 47p, Capacitor_SMD:C_0603_1608Metric, symbol Device:C
- removed C60: 220uF 25V, Capacitor_SMD:CP_Elec_6.3x7.7, symbol Device:C_Polarized
- removed D15: SMAJ51A, Diode_SMD:D_SMC, symbol Diode:SMF54A
- removed D16: SS310, Diode_SMD:D_SMA, symbol Diode:MBR340
- removed F1: 60V 1.5A hold polyfuse, Fuse:Fuse_2920_7451Metric, symbol Device:Polyfuse
- removed L1: 47uH, Inductor_SMD:L_Chilisin_BMRB00060612, symbol Device:L
- removed L3: 68uH 1A, Inductor_SMD:L_Sunlord_SWPA6045S, symbol Device:L
- removed R56: 30mΩ 5%, Resistor_SMD:R_0603_1608Metric, symbol Device:R
- removed R57: 10Ω, Resistor_SMD:R_0603_1608Metric, symbol Device:R
- removed R58: 300k, Resistor_SMD:R_0603_1608Metric, symbol Device:R
- removed R59: 21.5k, Resistor_SMD:R_0603_1608Metric, symbol Device:R
- removed U13: TX4139, Package_SO:SOIC-8-1EP_3.9x4.9mm_P1.27mm_EP2.29x3mm_ThermalVias, symbol MotorBuck:TX4139
Other:
- note removed: "52 Volt input max"
- note removed: "Internal pullup on EN"
- note removed: "Pi filter with ~18khz cutoff frequency"
- note removed: "R_{ILIM} 30mohm = 2A Iout max"
