File: BaselineRP2040MotorController/BaselineRP2040MotorController.kicad_pcb (KiCad board)
At the start: 2 copper layers, 75 x 75 mm, 106 parts, among them J2 Encoder 1, J3 3 Pin XT30 / XT60, J4 XT60 Power Connector, J5 Conn_02x08_Odd_Even, U10 INA240A1D, U11 USBLC6-4SC6, U13 TX4139, U5 EG3113, U6 INA240A1D, U7 EG3113, U8 INA240A1D, U9 EG3113

Commit message: Generate Gerbers
Parts:
- added REF**: EastMakesLogo1x2CM, [EastMakes]BrandingLibrary:EastMakesLogo1x2CM, F.Cu at (121.9, 98.6)
Routing:
- net /CurrentSense3: track 48.0 -> 47.5 mm, vias 5 -> 4
- net +3V3: track 156.3 -> 155.9 mm, vias 12 -> 11
Other:
- outline, holes or cut-outs redrawn
- board text added: "BLDC Test Board"
