File: BaselineRP2040MotorController/BLDC_Power_Control/BLDC_Motor_Phase.kicad_sch (KiCad schematic)
At the start: 16 parts, among them U9 EG3113

Commit message: Heh - Super cut down.
Parts:
- removed R38, R39, R40: 0R, Resistor_SMD:R_0603_1608Metric, symbol MotorController:TAYLOR_RESISTOR
Connections:
- net at R43.1, U9.5 (LO): now also D12.1 (K)
- net at D10.1 (K): now also C32.2, U9.8 (VB)
- net at D11.1 (K): now also R42.1, U9.7 (HO)
